File: eagle/schematic.brd (EAGLE design)
At the start: 44.1 x 45.7 mm, 35 parts, among them U1 PIC18F252-I/SP

Commit message: Corrigé les bugs restants, mis à jour la documentation
Connections:
- net HR1: now also U1.26; no longer U1.6
Routing:
- net HR1: track 28.8 -> 24.1 mm
Other:
- board text added: "2017-01-07 Version 1.0.0"
- board text removed: "2016-11-27 Version 0.1.1"
Changed lines of the file:
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@@
 <hole x="40.9575" y="42.545" drill="3.2"/>
 <hole x="14.605" y="3.81" drill="3.2"/>
-<text x="33.02" y="38.735" size="0.6096" layer="25">2016-11-27
-Version 0.1.1</text>
+<text x="33.02" y="38.735" size="0.6096" layer="25">2017-01-07
+Version 1.0.0</text>
 <polygon width="0.4064" layer="25">
 <vertex x="19.05" y="41.275"/>
@@
 </signal>
 <signal name="HR1">
-<contactref element="U1" pad="6"/>
 <contactref element="R6" pad="P$2"/>
 <wire x1="15.875" y1="40.005" x2="21.59" y2="40.005" width="0.254" layer="1"/>
@@
 <wire x1="22.5425" y1="39.0525" x2="24.13" y2="39.0525" width="0.254" layer="1"/>
 <via x="24.13" y="39.0525" extent="1-16" drill="0.6096" shape="square"/>
-<wire x1="24.13" y1="39.0525" x2="24.13" y2="26.67" width="0.254" layer="16"/>
-<wire x1="24.13" y1="26.67" x2="22.86" y2="25.4" width="0.254" layer="16"/>
-<via x="22.86" y="25.4" extent="1-16" drill="0.6096" shape="square"/>
-<wire x1="22.86" y1="25.4" x2="20.32" y2="22.86" width="0.254" layer="1"/>
-<wire x1="20.32" y1="22.86" x2="20.066" y2="22.86" width="0.254" layer="1"/>
+<wire x1="24.13" y1="39.0525" x2="24.13" y2="29.845" width="0.254" layer="16"/>
+<via x="24.13" y="29.845" extent="1-16" drill="0.6096" shape="square"/>
 <wire x1="15.875" y1="40.005" x2="15.24" y2="40.64" width="0.2032" layer="1"/>
 <wire x1="15.24" y1="40.64" x2="13.97" y2="40.64" width="0.2032" layer="1"/>
+<contactref element="U1" pad="26"/>
+<wire x1="24.13" y1="29.845" x2="27.305" y2="29.845" width="0.2032" layer="1"/>
+<wire x1="27.305" y1="29.845" x2="27.94" y2="30.48" width="0.2032" layer="1"/>
 </signal>
 <signal name="HR2">
